Commit message: Add functional SCARA gripper and expanded pickup scene

File: ros2_ws/src/scara_description/urdf/scara.urdf.xacro (robot description, xacro)
@@ -8,5 +8,5 @@
 <joint name="world_fixed" type="fixed"><parent link="world"/><child link="base_link"/></joint>
 <link name="base_link">
-<visual><geometry><mesh filename="file://$(arg description_share)/meshes/base_link.stl"/></geometry><material name="base_link_color"><color rgba="0.18 0.22 0.28 1"/></material></visual>
+<visual><geometry><mesh filename="file://$(arg description_share)/meshes/base_link.stl"/></geometry><material name="base_link_color"><color rgba="0.02 0.28 0.82 1"/></material></visual>
 <collision><geometry><mesh filename="file://$(arg description_share)/meshes/base_link_collision_000.stl"/></geometry></collision>
 <collision><geometry><mesh filename="file://$(arg description_share)/meshes/base_link_collision_001.stl"/></geometry></collision>
@@ -30,5 +30,5 @@
 </link>
 <link name="arm1_link">
-<visual><geometry><mesh filename="file://$(arg description_share)/meshes/arm1_link.stl"/></geometry><material name="arm1_link_color"><color rgba="0.10 0.50 0.68 1"/></material></visual>
+<visual><geometry><mesh filename="file://$(arg description_share)/meshes/arm1_link.stl"/></geometry><material name="arm1_link_color"><color rgba="0.02 0.28 0.82 1"/></material></visual>
 <collision><geometry><mesh filename="file://$(arg description_share)/meshes/arm1_link_collision_028.stl"/></geometry></collision>
 <collision><geometry><mesh filename="file://$(arg description_share)/meshes/arm1_link_collision_029.stl"/></geometry></collision>
@@ -38,5 +38,5 @@
 </link>
 <link name="arm2_link">
-<visual><geometry><mesh filename="file://$(arg description_share)/meshes/arm2_link.stl"/></geometry><material name="arm2_link_color"><color rgba="0.10 0.50 0.68 1"/></material></visual>
+<visual><geometry><mesh filename="file://$(arg description_share)/meshes/arm2_link.stl"/></geometry><material name="arm2_link_color"><color rgba="0.02 0.28 0.82 1"/></material></visual>
 <collision><geometry><mesh filename="file://$(arg description_share)/meshes/arm2_link_collision_032.stl"/></geometry></collision>
 <collision><geometry><mesh filename="file://$(arg description_share)/meshes/arm2_link_collision_045.stl"/></geometry></collision>
@@ -46,5 +46,5 @@
 </link>
 <link name="tool_link">
-<visual><geometry><mesh filename="file://$(arg description_share)/meshes/tool_link.stl"/></geometry><material name="tool_link_color"><color rgba="0.30 0.34 0.40 1"/></material></visual>
+<visual><geometry><mesh filename="file://$(arg description_share)/meshes/tool_link.stl"/></geometry><material name="tool_link_color"><color rgba="0.95 0.95 0.95 1"/></material></visual>
 <collision><geometry><mesh filename="file://$(arg description_share)/meshes/tool_link_collision_049.stl"/></geometry></collision>
 <collision><geometry><mesh filename="file://$(arg description_share)/meshes/tool_link_collision_058.stl"/></geometry></collision>
@@ -64,10 +64,28 @@
 <inertial><origin xyz="2.949029909160572e-15 -5.304784389537076e-15 -0.03533070698027093"/><mass value="0.35"/><inertia ixx="0.0010352714832298565" ixy="0" ixz="0" iyy="0.0010119555516648687" iyz="0" izz="0.0005639303865941157"/></inertial>
 </link>
-<joint name="shoulder_joint" type="revolute"><parent link="base_link"/><child link="shoulder_link"/><origin xyz="0 0 0.066"/><axis xyz="0 0 1"/><limit lower="-1.5707963267948966" upper="4.642575810304916" effort="10" velocity="0.5"/><dynamics damping="0.1" friction="0.01"/></joint>
-<joint name="z_joint" type="prismatic"><parent link="shoulder_link"/><child link="arm1_link"/><origin xyz="0 0 0.19761649586021549"/><axis xyz="0 0 1"/><limit lower="-0.05" upper="0.05" effort="100" velocity="0.02"/><dynamics damping="0.1" friction="0.01"/></joint>
-<joint name="elbow_joint" type="revolute"><parent link="arm1_link"/><child link="arm2_link"/><origin xyz="0.22799999999999893 0 -0.01899999999999869"/><axis xyz="0 0 1"/><limit lower="-2.6179938779914944" upper="2.6179938779914944" effort="10" velocity="0.6"/><dynamics damping="0.1" friction="0.01"/></joint>
-<joint name="wrist_joint" type="revolute"><parent link="arm2_link"/><child link="tool_link"/><origin xyz="0.13649999999995294 0 -0.0570000000000017"/><axis xyz="0 0 1"/><limit lower="-2.827433388230814" upper="2.827433388230814" effort="10" velocity="1.0"/><dynamics damping="0.1" friction="0.01"/></joint>
+<joint name="shoulder_joint" type="revolute"><parent link="base_link"/><child link="shoulder_link"/><origin xyz="0 0 0.066"/><axis xyz="0 0 1"/><limit lower="-1.5707963267948966" upper="4.642575810304916" effort="20" velocity="1.2"/><dynamics damping="0.1" friction="0.01"/></joint>
+<joint name="z_joint" type="prismatic"><parent link="shoulder_link"/><child link="arm1_link"/><origin xyz="0 0 0.19761649586021549"/><axis xyz="0 0 1"/><limit lower="-0.05" upper="0.05" effort="150" velocity="0.08"/><dynamics damping="0.1" friction="0.01"/></joint>
+<joint name="elbow_joint" type="revolute"><parent link="arm1_link"/><child link="arm2_link"/><origin xyz="0.22799999999999893 0 -0.01899999999999869"/><axis xyz="0 0 1"/><limit lower="-2.6179938779914944" upper="2.6179938779914944" effort="20" velocity="1.5"/><dynamics damping="0.1" friction="0.01"/></joint>
+<joint name="wrist_joint" type="revolute"><parent link="arm2_link"/><child link="tool_link"/><origin xyz="0.13649999999995294 0 -0.0570000000000017"/><axis xyz="0 0 1"/><limit lower="-2.827433388230814" upper="2.827433388230814" effort="15" velocity="2.0"/><dynamics damping="0.1" friction="0.01"/></joint>
 <link name="tcp_link"/>
 <joint name="tcp_fixed" type="fixed"><parent link="tool_link"/><child link="tcp_link"/><origin xyz="0 0 -0.11506141396054323"/></joint>
+<link name="gripper_base_link">
+<visual><origin xyz="0 0 -0.008"/><geometry><box size="0.050 0.070 0.016"/></geometry><material name="gripper_white"><color rgba="0.96 0.96 0.96 1"/></material></visual>
+<collision><origin xyz="0 0 -0.008"/><geometry><box size="0.050 0.070 0.016"/></geometry></collision>
+<inertial><origin xyz="0 0 -0.008"/><mass value="0.10"/><inertia ixx="0.000044" ixy="0" ixz="0" iyy="0.000023" iyz="0" izz="0.000061"/></inertial>
+</link>
+<joint name="gripper_base_fixed" type="fixed"><parent link="tool_link"/><child link="gripper_base_link"/><origin xyz="0 0 -0.052"/></joint>
+<link name="left_finger_link">
+<visual><origin xyz="0 0 -0.033"/><geometry><box size="0.018 0.012 0.066"/></geometry><material name="finger_white"><color rgba="1 1 1 1"/></material></visual>
+<collision><origin xyz="0 0 -0.033"/><geometry><box size="0.018 0.012 0.066"/></geometry></collision>
+<inertial><origin xyz="0 0 -0.033"/><mass value="0.035"/><inertia ixx="0.000013" ixy="0" ixz="0" iyy="0.000014" iyz="0" izz="0.000002"/></inertial>
+</link>
+<link name="right_finger_link">
+<visual><origin xyz="0 0 -0.033"/><geometry><box size="0.018 0.012 0.066"/></geometry><material name="finger_white"><color rgba="1 1 1 1"/></material></visual>
+<collision><origin xyz="0 0 -0.033"/><geometry><box size="0.018 0.012 0.066"/></geometry></collision>
+<inertial><origin xyz="0 0 -0.033"/><mass value="0.035"/><inertia ixx="0.000013" ixy="0" ixz="0" iyy="0.000014" iyz="0" izz="0.000002"/></inertial>
+</link>
+<joint name="left_finger_joint" type="prismatic"><parent link="gripper_base_link"/><child link="left_finger_link"/><origin xyz="0 0.022 0"/><axis xyz="0 1 0"/><limit lower="0" upper="0.025" effort="40" velocity="0.08"/><dynamics damping="0.2" friction="0.02"/></joint>
+<joint name="right_finger_joint" type="prismatic"><parent link="gripper_base_link"/><child link="right_finger_link"/><origin xyz="0 -0.022 0"/><axis xyz="0 -1 0"/><limit lower="0" upper="0.025" effort="40" velocity="0.08"/><dynamics damping="0.2" friction="0.02"/></joint>
 <ros2_control name="ScaraSystem" type="system"><hardware>
 <xacro:if value="${mode == 'gazebo'}"><plugin>gazebo_ros2_control/GazeboSystem</plugin></xacro:if>
@@ -78,12 +96,18 @@
 <joint name="elbow_joint"><command_interface name="position"/><state_interface name="position"><param name="initial_value">0.0</param></state_interface><state_interface name="velocity"/></joint>
 <joint name="wrist_joint"><command_interface name="position"/><state_interface name="position"><param name="initial_value">0.0</param></state_interface><state_interface name="velocity"/></joint>
+<joint name="left_finger_joint"><command_interface name="position"/><state_interface name="position"><param name="initial_value">0.025</param></state_interface><state_interface name="velocity"/></joint>
+<joint name="right_finger_joint"><command_interface name="position"/><state_interface name="position"><param name="initial_value">0.025</param></state_interface><state_interface name="velocity"/></joint>
 </ros2_control>
 <xacro:if value="${mode == 'gazebo'}">
 <gazebo><plugin name="gazebo_ros2_control" filename="libgazebo_ros2_control.so"><robot_param>robot_description</robot_param><robot_param_node>robot_state_publisher</robot_param_node><parameters>$(arg controllers_file)</parameters></plugin></gazebo>
-<gazebo reference="base_link"><selfCollide>false</selfCollide><material>Gazebo/Grey</material></gazebo>
+<gazebo reference="base_link"><selfCollide>false</selfCollide><material>Gazebo/Blue</material></gazebo>
 <gazebo reference="shoulder_link"><selfCollide>false</selfCollide><material>Gazebo/Grey</material></gazebo>
 <gazebo reference="arm1_link"><selfCollide>false</selfCollide><material>Gazebo/Blue</material></gazebo>
 <gazebo reference="arm2_link"><selfCollide>false</selfCollide><material>Gazebo/Blue</material></gazebo>
-<gazebo reference="tool_link"><selfCollide>false</selfCollide><material>Gazebo/Grey</material></gazebo>
+<gazebo reference="tool_link"><selfCollide>false</selfCollide><material>Gazebo/White</material></gazebo>
+<gazebo reference="gripper_base_link"><selfCollide>false</selfCollide><material>Gazebo/White</material></gazebo>
+<gazebo reference="left_finger_link"><selfCollide>false</selfCollide><material>Gazebo/White</material></gazebo>
+<gazebo reference="right_finger_link"><selfCollide>false</selfCollide><material>Gazebo/White</material></gazebo>
+<gazebo><plugin name="scara_grasp" filename="libscara_grasp_plugin.so"><gripper_link>gripper_base_link</gripper_link><left_joint>left_finger_joint</left_joint><right_joint>right_finger_joint</right_joint><attach_distance>0.072</attach_distance><closed_threshold>0.006</closed_threshold><open_threshold>0.016</open_threshold><targets>pickup_cube pickup_sphere pickup_cylinder pickup_hex_prism hanoi_ring_large hanoi_ring_medium hanoi_ring_small</targets></plugin></gazebo>
 </xacro:if>
 </robot>

Commit message: Fix duplicate SCARA gripper visual and increase joint speeds

File: ros2_ws/src/scara_description/urdf/scara.urdf.xacro (robot description, xacro)
@@ -46,5 +46,5 @@
 </link>
 <link name="tool_link">
-<visual><geometry><mesh filename="file://$(arg description_share)/meshes/tool_link.stl"/></geometry><material name="tool_link_color"><color rgba="0.95 0.95 0.95 1"/></material></visual>
+<visual><origin xyz="0 0 -0.010"/><geometry><cylinder radius="0.028" length="0.020"/></geometry><material name="tool_link_color"><color rgba="0.95 0.95 0.95 1"/></material></visual>
 <collision><geometry><mesh filename="file://$(arg description_share)/meshes/tool_link_collision_049.stl"/></geometry></collision>
 <collision><geometry><mesh filename="file://$(arg description_share)/meshes/tool_link_collision_058.stl"/></geometry></collision>
@@ -64,8 +64,8 @@
 <inertial><origin xyz="2.949029909160572e-15 -5.304784389537076e-15 -0.03533070698027093"/><mass value="0.35"/><inertia ixx="0.0010352714832298565" ixy="0" ixz="0" iyy="0.0010119555516648687" iyz="0" izz="0.0005639303865941157"/></inertial>
 </link>
-<joint name="shoulder_joint" type="revolute"><parent link="base_link"/><child link="shoulder_link"/><origin xyz="0 0 0.066"/><axis xyz="0 0 1"/><limit lower="-1.5707963267948966" upper="4.642575810304916" effort="20" velocity="1.2"/><dynamics damping="0.1" friction="0.01"/></joint>
-<joint name="z_joint" type="prismatic"><parent link="shoulder_link"/><child link="arm1_link"/><origin xyz="0 0 0.19761649586021549"/><axis xyz="0 0 1"/><limit lower="-0.05" upper="0.05" effort="150" velocity="0.08"/><dynamics damping="0.1" friction="0.01"/></joint>
-<joint name="elbow_joint" type="revolute"><parent link="arm1_link"/><child link="arm2_link"/><origin xyz="0.22799999999999893 0 -0.01899999999999869"/><axis xyz="0 0 1"/><limit lower="-2.6179938779914944" upper="2.6179938779914944" effort="20" velocity="1.5"/><dynamics damping="0.1" friction="0.01"/></joint>
-<joint name="wrist_joint" type="revolute"><parent link="arm2_link"/><child link="tool_link"/><origin xyz="0.13649999999995294 0 -0.0570000000000017"/><axis xyz="0 0 1"/><limit lower="-2.827433388230814" upper="2.827433388230814" effort="15" velocity="2.0"/><dynamics damping="0.1" friction="0.01"/></joint>
+<joint name="shoulder_joint" type="revolute"><parent link="base_link"/><child link="shoulder_link"/><origin xyz="0 0 0.066"/><axis xyz="0 0 1"/><limit lower="-1.5707963267948966" upper="4.642575810304916" effort="20" velocity="2.4"/><dynamics damping="0.1" friction="0.01"/></joint>
+<joint name="z_joint" type="prismatic"><parent link="shoulder_link"/><child link="arm1_link"/><origin xyz="0 0 0.19761649586021549"/><axis xyz="0 0 1"/><limit lower="-0.05" upper="0.05" effort="150" velocity="0.16"/><dynamics damping="0.1" friction="0.01"/></joint>
+<joint name="elbow_joint" type="revolute"><parent link="arm1_link"/><child link="arm2_link"/><origin xyz="0.22799999999999893 0 -0.01899999999999869"/><axis xyz="0 0 1"/><limit lower="-2.6179938779914944" upper="2.6179938779914944" effort="20" velocity="3.0"/><dynamics damping="0.1" friction="0.01"/></joint>
+<joint name="wrist_joint" type="revolute"><parent link="arm2_link"/><child link="tool_link"/><origin xyz="0.13649999999995294 0 -0.0570000000000017"/><axis xyz="0 0 1"/><limit lower="-2.827433388230814" upper="2.827433388230814" effort="15" velocity="4.0"/><dynamics damping="0.1" friction="0.01"/></joint>
 <link name="tcp_link"/>
 <joint name="tcp_fixed" type="fixed"><parent link="tool_link"/><child link="tcp_link"/><origin xyz="0 0 -0.11506141396054323"/></joint>
@@ -86,6 +86,6 @@
 <inertial><origin xyz="0 0 -0.033"/><mass value="0.035"/><inertia ixx="0.000013" ixy="0" ixz="0" iyy="0.000014" iyz="0" izz="0.000002"/></inertial>
 </link>
-<joint name="left_finger_joint" type="prismatic"><parent link="gripper_base_link"/><child link="left_finger_link"/><origin xyz="0 0.022 0"/><axis xyz="0 1 0"/><limit lower="0" upper="0.025" effort="40" velocity="0.08"/><dynamics damping="0.2" friction="0.02"/></joint>
-<joint name="right_finger_joint" type="prismatic"><parent link="gripper_base_link"/><child link="right_finger_link"/><origin xyz="0 -0.022 0"/><axis xyz="0 -1 0"/><limit lower="0" upper="0.025" effort="40" velocity="0.08"/><dynamics damping="0.2" friction="0.02"/></joint>
+<joint name="left_finger_joint" type="prismatic"><parent link="gripper_base_link"/><child link="left_finger_link"/><origin xyz="0 0.022 0"/><axis xyz="0 1 0"/><limit lower="0" upper="0.025" effort="40" velocity="0.16"/><dynamics damping="0.2" friction="0.02"/></joint>
+<joint name="right_finger_joint" type="prismatic"><parent link="gripper_base_link"/><child link="right_finger_link"/><origin xyz="0 -0.022 0"/><axis xyz="0 -1 0"/><limit lower="0" upper="0.025" effort="40" velocity="0.16"/><dynamics damping="0.2" friction="0.02"/></joint>
 <ros2_control name="ScaraSystem" type="system"><hardware>
 <xacro:if value="${mode == 'gazebo'}"><plugin>gazebo_ros2_control/GazeboSystem</plugin></xacro:if>

Commit message: Remove hidden legacy gripper collision geometry

File: ros2_ws/src/scara_description/urdf/scara.urdf.xacro (robot description, xacro)
@@ -50,16 +50,4 @@
 <collision><geometry><mesh filename="file://$(arg description_share)/meshes/tool_link_collision_058.stl"/></geometry></collision>
 <collision><geometry><mesh filename="file://$(arg description_share)/meshes/tool_link_collision_059.stl"/></geometry></collision>
-<collision><geometry><mesh filename="file://$(arg description_share)/meshes/tool_link_collision_061.stl"/></geometry></collision>
-<collision><geometry><mesh filename="file://$(arg description_share)/meshes/tool_link_collision_062.stl"/></geometry></collision>
-<collision><geometry><mesh filename="file://$(arg description_share)/meshes/tool_link_collision_063.stl"/></geometry></collision>
-<collision><geometry><mesh filename="file://$(arg description_share)/meshes/tool_link_collision_064.stl"/></geometry></collision>
-<collision><geometry><mesh filename="file://$(arg description_share)/meshes/tool_link_collision_065.stl"/></geometry></collision>
-<collision><geometry><mesh filename="file://$(arg description_share)/meshes/tool_link_collision_066.stl"/></geometry></collision>
-<collision><geometry><mesh filename="file://$(arg description_share)/meshes/tool_link_collision_067.stl"/></geometry></collision>
-<collision><geometry><mesh filename="file://$(arg description_share)/meshes/tool_link_collision_068.stl"/></geometry></collision>
-<collision><geometry><mesh filename="file://$(arg description_share)/meshes/tool_link_collision_069.stl"/></geometry></collision>
-<collision><geometry><mesh filename="file://$(arg description_share)/meshes/tool_link_collision_070.stl"/></geometry></collision>
-<collision><geometry><mesh filename="file://$(arg description_share)/meshes/tool_link_collision_071.stl"/></geometry></collision>
-<collision><geometry><mesh filename="file://$(arg description_share)/meshes/tool_link_collision_076.stl"/></geometry></collision>
 <inertial><origin xyz="2.949029909160572e-15 -5.304784389537076e-15 -0.03533070698027093"/><mass value="0.35"/><inertia ixx="0.0010352714832298565" ixy="0" ixz="0" iyy="0.0010119555516648687" iyz="0" izz="0.0005639303865941157"/></inertial>
 </link>
