Commit message: Animate original CAD-derived SCARA gripper jaws

File: ros2_ws/src/scara_description/urdf/scara.urdf.xacro (robot description, xacro)
@@ -46,9 +46,11 @@
 </link>
 <link name="tool_link">
-<visual><origin xyz="0 0 -0.010"/><geometry><cylinder radius="0.028" length="0.020"/></geometry><material name="tool_link_color"><color rgba="0.95 0.95 0.95 1"/></material></visual>
-<collision><geometry><mesh filename="file://$(arg description_share)/meshes/tool_link_collision_049.stl"/></geometry></collision>
-<collision><geometry><mesh filename="file://$(arg description_share)/meshes/tool_link_collision_058.stl"/></geometry></collision>
-<collision><geometry><mesh filename="file://$(arg description_share)/meshes/tool_link_collision_059.stl"/></geometry></collision>
-<inertial><origin xyz="2.949029909160572e-15 -5.304784389537076e-15 -0.03533070698027093"/><mass value="0.35"/><inertia ixx="0.0010352714832298565" ixy="0" ixz="0" iyy="0.0010119555516648687" iyz="0" izz="0.0005639303865941157"/></inertial>
+  <visual><geometry><mesh filename="file://$(arg description_share)/meshes/tool_link_collision_049.stl"/></geometry><material name="tool_link_white"><color rgba="0.95 0.95 0.95 1"/></material></visual>
+  <visual><geometry><mesh filename="file://$(arg description_share)/meshes/tool_link_collision_058.stl"/></geometry><material name="tool_link_white_2"><color rgba="0.95 0.95 0.95 1"/></material></visual>
+  <visual><geometry><mesh filename="file://$(arg description_share)/meshes/tool_link_collision_059.stl"/></geometry><material name="tool_link_white_3"><color rgba="0.95 0.95 0.95 1"/></material></visual>
+  <collision><geometry><mesh filename="file://$(arg description_share)/meshes/tool_link_collision_049.stl"/></geometry></collision>
+  <collision><geometry><mesh filename="file://$(arg description_share)/meshes/tool_link_collision_058.stl"/></geometry></collision>
+  <collision><geometry><mesh filename="file://$(arg description_share)/meshes/tool_link_collision_059.stl"/></geometry></collision>
+  <inertial><origin xyz="2.949029909160572e-15 -5.304784389537076e-15 -0.03533070698027093"/><mass value="0.35"/><inertia ixx="0.0010352714832298565" ixy="0" ixz="0" iyy="0.0010119555516648687" iyz="0" izz="0.0005639303865941157"/></inertial>
 </link>
 <joint name="shoulder_joint" type="revolute"><parent link="base_link"/><child link="shoulder_link"/><origin xyz="0 0 0.066"/><axis xyz="0 0 1"/><limit lower="-1.5707963267948966" upper="4.642575810304916" effort="20" velocity="2.4"/><dynamics damping="0.1" friction="0.01"/></joint>
@@ -59,21 +61,57 @@
 <joint name="tcp_fixed" type="fixed"><parent link="tool_link"/><child link="tcp_link"/><origin xyz="0 0 -0.11506141396054323"/></joint>
 <link name="gripper_base_link">
-<visual><origin xyz="0 0 -0.008"/><geometry><box size="0.050 0.070 0.016"/></geometry><material name="gripper_white"><color rgba="0.96 0.96 0.96 1"/></material></visual>
-<collision><origin xyz="0 0 -0.008"/><geometry><box size="0.050 0.070 0.016"/></geometry></collision>
-<inertial><origin xyz="0 0 -0.008"/><mass value="0.10"/><inertia ixx="0.000044" ixy="0" ixz="0" iyy="0.000023" iyz="0" izz="0.000061"/></inertial>
+  <!-- Static pieces from the original SCARA gripper CAD: cover, rails and J3 connector. -->
+  <visual><geometry><mesh filename="file://$(arg description_share)/meshes/tool_link_collision_061.stl"/></geometry><material name="gripper_cad_white"><color rgba="1 1 1 1"/></material></visual>
+  <visual><geometry><mesh filename="file://$(arg description_share)/meshes/tool_link_collision_063.stl"/></geometry><material name="gripper_cad_white_2"><color rgba="1 1 1 1"/></material></visual>
+  <visual><geometry><mesh filename="file://$(arg description_share)/meshes/tool_link_collision_066.stl"/></geometry><material name="gripper_cad_white_3"><color rgba="1 1 1 1"/></material></visual>
+  <visual><geometry><mesh filename="file://$(arg description_share)/meshes/tool_link_collision_076.stl"/></geometry><material name="gripper_cad_white_4"><color rgba="1 1 1 1"/></material></visual>
+  <collision><geometry><mesh filename="file://$(arg description_share)/meshes/tool_link_collision_061.stl"/></geometry></collision>
+  <collision><geometry><mesh filename="file://$(arg description_share)/meshes/tool_link_collision_063.stl"/></geometry></collision>
+  <collision><geometry><mesh filename="file://$(arg description_share)/meshes/tool_link_collision_066.stl"/></geometry></collision>
+  <collision><geometry><mesh filename="file://$(arg description_share)/meshes/tool_link_collision_076.stl"/></geometry></collision>
+  <inertial><mass value="0.10"/><inertia ixx="0.000044" ixy="0" ixz="0" iyy="0.000023" iyz="0" izz="0.000061"/></inertial>
 </link>
-<joint name="gripper_base_fixed" type="fixed"><parent link="tool_link"/><child link="gripper_base_link"/><origin xyz="0 0 -0.052"/></joint>
+<joint name="gripper_base_fixed" type="fixed"><parent link="tool_link"/><child link="gripper_base_link"/><origin xyz="0 0 0"/></joint>
 <link name="left_finger_link">
-<visual><origin xyz="0 0 -0.033"/><geometry><box size="0.018 0.012 0.066"/></geometry><material name="finger_white"><color rgba="1 1 1 1"/></material></visual>
-<collision><origin xyz="0 0 -0.033"/><geometry><box size="0.018 0.012 0.066"/></geometry></collision>
-<inertial><origin xyz="0 0 -0.033"/><mass value="0.035"/><inertia ixx="0.000013" ixy="0" ixz="0" iyy="0.000014" iyz="0" izz="0.000002"/></inertial>
+  <!-- Original CAD left jaw assembly.  Meshes are expressed in tool coordinates;
+       the visual/collision offset preserves the source CAD OPEN pose at q=0.025 m. -->
+  <visual><origin xyz="0.032307 0.034136 0"/><geometry><mesh filename="file://$(arg description_share)/meshes/tool_link_collision_062.stl"/></geometry><material name="left_cad_white"><color rgba="1 1 1 1"/></material></visual>
+  <visual><origin xyz="0.032307 0.034136 0"/><geometry><mesh filename="file://$(arg description_share)/meshes/tool_link_collision_064.stl"/></geometry><material name="left_cad_white_2"><color rgba="1 1 1 1"/></material></visual>
+  <visual><origin xyz="0.032307 0.034136 0"/><geometry><mesh filename="file://$(arg description_share)/meshes/tool_link_collision_067.stl"/></geometry><material name="left_cad_white_3"><color rgba="1 1 1 1"/></material></visual>
+  <visual><origin xyz="0.032307 0.034136 0"/><geometry><mesh filename="file://$(arg description_share)/meshes/tool_link_collision_069.stl"/></geometry><material name="left_cad_white_4"><color rgba="1 1 1 1"/></material></visual>
+  <collision><origin xyz="0.032307 0.034136 0"/><geometry><mesh filename="file://$(arg description_share)/meshes/tool_link_collision_062.stl"/></geometry></collision>
+  <collision><origin xyz="0.032307 0.034136 0"/><geometry><mesh filename="file://$(arg description_share)/meshes/tool_link_collision_064.stl"/></geometry></collision>
+  <collision><origin xyz="0.032307 0.034136 0"/><geometry><mesh filename="file://$(arg description_share)/meshes/tool_link_collision_067.stl"/></geometry></collision>
+  <collision><origin xyz="0.032307 0.034136 0"/><geometry><mesh filename="file://$(arg description_share)/meshes/tool_link_collision_069.stl"/></geometry></collision>
+  <inertial><mass value="0.060"/><inertia ixx="0.000020" ixy="0" ixz="0" iyy="0.000020" iyz="0" izz="0.000006"/></inertial>
 </link>
 <link name="right_finger_link">
-<visual><origin xyz="0 0 -0.033"/><geometry><box size="0.018 0.012 0.066"/></geometry><material name="finger_white"><color rgba="1 1 1 1"/></material></visual>
-<collision><origin xyz="0 0 -0.033"/><geometry><box size="0.018 0.012 0.066"/></geometry></collision>
-<inertial><origin xyz="0 0 -0.033"/><mass value="0.035"/><inertia ixx="0.000013" ixy="0" ixz="0" iyy="0.000014" iyz="0" izz="0.000002"/></inertial>
+  <!-- Original CAD right jaw assembly. -->
+  <visual><origin xyz="-0.032307 -0.034136 0"/><geometry><mesh filename="file://$(arg description_share)/meshes/tool_link_collision_065.stl"/></geometry><material name="right_cad_white"><color rgba="1 1 1 1"/></material></visual>
+  <visual><origin xyz="-0.032307 -0.034136 0"/><geometry><mesh filename="file://$(arg description_share)/meshes/tool_link_collision_068.stl"/></geometry><material name="right_cad_white_2"><color rgba="1 1 1 1"/></material></visual>
+  <visual><origin xyz="-0.032307 -0.034136 0"/><geometry><mesh filename="file://$(arg description_share)/meshes/tool_link_collision_070.stl"/></geometry><material name="right_cad_white_3"><color rgba="1 1 1 1"/></material></visual>
+  <visual><origin xyz="-0.032307 -0.034136 0"/><geometry><mesh filename="file://$(arg description_share)/meshes/tool_link_collision_071.stl"/></geometry><material name="right_cad_white_4"><color rgba="1 1 1 1"/></material></visual>
+  <collision><origin xyz="-0.032307 -0.034136 0"/><geometry><mesh filename="file://$(arg description_share)/meshes/tool_link_collision_065.stl"/></geometry></collision>
+  <collision><origin xyz="-0.032307 -0.034136 0"/><geometry><mesh filename="file://$(arg description_share)/meshes/tool_link_collision_068.stl"/></geometry></collision>
+  <collision><origin xyz="-0.032307 -0.034136 0"/><geometry><mesh filename="file://$(arg description_share)/meshes/tool_link_collision_070.stl"/></geometry></collision>
+  <collision><origin xyz="-0.032307 -0.034136 0"/><geometry><mesh filename="file://$(arg description_share)/meshes/tool_link_collision_071.stl"/></geometry></collision>
+  <inertial><mass value="0.060"/><inertia ixx="0.000020" ixy="0" ixz="0" iyy="0.000020" iyz="0" izz="0.000006"/></inertial>
 </link>
-<joint name="left_finger_joint" type="prismatic"><parent link="gripper_base_link"/><child link="left_finger_link"/><origin xyz="0 0.022 0"/><axis xyz="0 1 0"/><limit lower="0" upper="0.025" effort="40" velocity="0.16"/><dynamics damping="0.2" friction="0.02"/></joint>
-<joint name="right_finger_joint" type="prismatic"><parent link="gripper_base_link"/><child link="right_finger_link"/><origin xyz="0 -0.022 0"/><axis xyz="0 -1 0"/><limit lower="0" upper="0.025" effort="40" velocity="0.16"/><dynamics damping="0.2" friction="0.02"/></joint>
+<!-- Parallel-jaw motion follows the actual slider axis measured from the source CAD.
+     q=0.025 m = source/open pose; q=0 = jaws translated 25 mm inward each. -->
+<joint name="left_finger_joint" type="prismatic">
+  <parent link="gripper_base_link"/><child link="left_finger_link"/>
+  <origin xyz="-0.015122 -0.015979 0"/>
+  <axis xyz="-0.687379 -0.726299 0"/>
+  <limit lower="0" upper="0.025" effort="40" velocity="0.16"/>
+  <dynamics damping="0.2" friction="0.02"/>
+</joint>
+<joint name="right_finger_joint" type="prismatic">
+  <parent link="gripper_base_link"/><child link="right_finger_link"/>
+  <origin xyz="0.015122 0.015979 0"/>
+  <axis xyz="0.687379 0.726299 0"/>
+  <limit lower="0" upper="0.025" effort="40" velocity="0.16"/>
+  <dynamics damping="0.2" friction="0.02"/>
+</joint>
 <ros2_control name="ScaraSystem" type="system"><hardware>
 <xacro:if value="${mode == 'gazebo'}"><plugin>gazebo_ros2_control/GazeboSystem</plugin></xacro:if>

Commit message: Use synchronized mimic motion for CAD gripper

File: ros2_ws/src/scara_description/urdf/scara.urdf.xacro (robot description, xacro)
@@ -105,4 +105,5 @@
   <origin xyz="0.015122 0.015979 0"/>
   <axis xyz="0.687379 0.726299 0"/>
+  <mimic joint="left_finger_joint" multiplier="1.0" offset="0.0"/>
   <limit lower="0" upper="0.025" effort="40" velocity="0.16"/>
   <dynamics damping="0.2" friction="0.02"/>
@@ -117,5 +118,5 @@
 <joint name="wrist_joint"><command_interface name="position"/><state_interface name="position"><param name="initial_value">0.0</param></state_interface><state_interface name="velocity"/></joint>
 <joint name="left_finger_joint"><command_interface name="position"/><state_interface name="position"><param name="initial_value">0.025</param></state_interface><state_interface name="velocity"/></joint>
-<joint name="right_finger_joint"><command_interface name="position"/><state_interface name="position"><param name="initial_value">0.025</param></state_interface><state_interface name="velocity"/></joint>
+<joint name="right_finger_joint"><param name="mimic">left_finger_joint</param><param name="multiplier">1.0</param><state_interface name="position"><param name="initial_value">0.025</param></state_interface><state_interface name="velocity"/></joint>
 </ros2_control>
 <xacro:if value="${mode == 'gazebo'}">

Commit message: Restore dual-joint CAD gripper control

File: ros2_ws/src/scara_description/urdf/scara.urdf.xacro (robot description, xacro)
@@ -105,5 +105,4 @@
   <origin xyz="0.015122 0.015979 0"/>
   <axis xyz="0.687379 0.726299 0"/>
-  <mimic joint="left_finger_joint" multiplier="1.0" offset="0.0"/>
   <limit lower="0" upper="0.025" effort="40" velocity="0.16"/>
   <dynamics damping="0.2" friction="0.02"/>
@@ -118,5 +117,5 @@
 <joint name="wrist_joint"><command_interface name="position"/><state_interface name="position"><param name="initial_value">0.0</param></state_interface><state_interface name="velocity"/></joint>
 <joint name="left_finger_joint"><command_interface name="position"/><state_interface name="position"><param name="initial_value">0.025</param></state_interface><state_interface name="velocity"/></joint>
-<joint name="right_finger_joint"><param name="mimic">left_finger_joint</param><param name="multiplier">1.0</param><state_interface name="position"><param name="initial_value">0.025</param></state_interface><state_interface name="velocity"/></joint>
+<joint name="right_finger_joint"><command_interface name="position"/><state_interface name="position"><param name="initial_value">0.025</param></state_interface><state_interface name="velocity"/></joint>
 </ros2_control>
 <xacro:if value="${mode == 'gazebo'}">
