Commit message: Assign Gazebo materials to STEP plates rods and motors

File: ros2_ws/src/scara_description/urdf/scara.urdf.xacro (robot description, xacro)
@@ -12,12 +12,4 @@
   </joint>
   <link name="base_link">
-    <visual>
-      <geometry>
-        <mesh filename="file://$(arg description_share)/meshes/base_link.stl"/>
-      </geometry>
-      <material name="base_link_color">
-        <color rgba="0.02 0.28 0.82 1"/>
-      </material>
-    </visual>
     <collision>
       <geometry>
@@ -47,9 +39,4 @@
   </link>
   <link name="shoulder_link">
-    <visual>
-      <geometry>
-        <mesh filename="file://$(arg description_share)/meshes/shoulder_colored.dae"/>
-      </geometry>
-    </visual>
     <collision>
       <geometry>
@@ -109,12 +96,4 @@
   </link>
   <link name="arm1_link">
-    <visual>
-      <geometry>
-        <mesh filename="file://$(arg description_share)/meshes/arm1_link.stl"/>
-      </geometry>
-      <material name="arm1_link_color">
-        <color rgba="0.02 0.28 0.82 1"/>
-      </material>
-    </visual>
     <collision>
       <geometry>
@@ -144,12 +123,4 @@
   </link>
   <link name="arm2_link">
-    <visual>
-      <geometry>
-        <mesh filename="file://$(arg description_share)/meshes/arm2_link.stl"/>
-      </geometry>
-      <material name="arm2_link_color">
-        <color rgba="0.02 0.28 0.82 1"/>
-      </material>
-    </visual>
     <collision>
       <geometry>
@@ -535,5 +506,4 @@
     <gazebo reference="base_link">
       <selfCollide>false</selfCollide>
-      <material>Gazebo/Blue</material>
     </gazebo>
     <gazebo reference="shoulder_link">
@@ -542,26 +512,24 @@
     <gazebo reference="arm1_link">
       <selfCollide>false</selfCollide>
-      <material>Gazebo/Blue</material>
     </gazebo>
     <gazebo reference="arm2_link">
       <selfCollide>false</selfCollide>
-      <material>Gazebo/Blue</material>
     </gazebo>
     <gazebo reference="tool_link">
       <selfCollide>false</selfCollide>
+    </gazebo>
+    <gazebo reference="gripper_base_link">
+      <selfCollide>false</selfCollide>
       <material>Gazebo/White</material>
     </gazebo>
-    <gazebo reference="gripper_base_link">
+    <gazebo reference="left_finger_link">
       <selfCollide>false</selfCollide>
       <material>Gazebo/White</material>
     </gazebo>
-    <gazebo reference="left_finger_link">
+    <gazebo reference="right_finger_link">
       <selfCollide>false</selfCollide>
       <material>Gazebo/White</material>
     </gazebo>
-    <gazebo reference="right_finger_link">
-      <selfCollide>false</selfCollide>
-      <material>Gazebo/White</material>
-    </gazebo>
   </xacro:if>
+  <xacro:include filename="$(arg description_share)/meshes/colored_visuals.xacro"/>
 </robot>
